File: PCB/CoreElectronics-Logic-Level-Converter-Bidirectional.kicad_pcb (KiCad board)
At the start: 2 copper layers, 15.2 x 12.7 mm, 18 parts, among them Q1 BSS138, Q2 BSS138, Q3 BSS138, Q4 BSS138

Commit message: update design with datamatrix
Parts:
- added G2: LOGO_made-with-love, datamatrix:CE07510, B.Cu at (10.2, 6.35)
- G1: footprint CoreElectronics_Logos:CoreElectronics_logo_5mm_v2 -> core-logo:core-logo
- moved G1 7.25 mm to (3.05, 5.21)
- moved LOGO1 3.08 mm to (2.92, 9.02)
Other:
- net class Default removed
- rule pad_to_mask_clearance: 0.05 -> 0
- board text removed: "logic level converter"
